File: ActivePrecharge.kicad_sch (KiCad schematic)
At the start: 52 parts, among them Con1 LED, IC1 1769205241, J1 Conn_01x03, J2 Conn_01x02, J3 Conn_02x03_Top_Bottom, J4 Conn_01x03, Q1 IRLML0030, Q3 IRLML0030, Q4 Q_PMOS_GDS, U3 TLV9301xDCK, U4 TCMT1106

Commit message: contactor board first revisions
Parts:
- removed J3: Conn_02x03_Top_Bottom, Active-PrechargeLib:CONN_SD-43045-005_06_MOL, symbol Connector_Generic:Conn_02x03_Top_Bottom
- removed J4: Conn_01x03, utsvt-conn:Molex_MicroFit3.0_1x3xP3.00mm_PolarizingPeg_Vertical, symbol Connector_Generic:Conn_01x03
- removed Q1: IRLML0030, Package_TO_SOT_SMD:SOT-23, symbol Transistor_FET:IRLML0030
- removed R6: 500k, Resistor_SMD:R_1206_3216Metric, symbol Device:R_US
- removed R7: 50k, Resistor_SMD:R_0805_2012Metric, symbol Device:R_US
- removed SigLV_TP1: TestPoint, utsvt-special:TestPoint_HEX_3mmID, symbol Connector:TestPoint
- added Con2: LED, LED_SMD:LED_0805_2012Metric, symbol Device:LED
- added D6: D, Active-PrechargeLib:SODFL4724X108N, symbol Device:D
- added J4, J5, J6, J7: Conn_01x04, utsvt-conn:Molex_MicroFit3.0_1x4xP3.00mm_PolarizingPeg_Vertical, symbol Connector_Generic:Conn_01x04
- added Q2: IRLML0030, Package_TO_SOT_SMD:SOT-23, symbol Transistor_FET:IRLML0030
- added R14, R16: 10k, Resistor_SMD:R_0805_2012Metric, symbol Device:R_US
- added R17: 1k, Resistor_SMD:R_0805_2012Metric, symbol Device:R_US
- added SignalLV1: TestPoint, utsvt-special:TestPoint_HEX_3mmID, symbol Connector:TestPoint
- added U1: Nucleo_L432KC, utsvt-special:NucleoL432KC, symbol utsvt-microcontrokller:Nucleo_L432KC
- R10: value 100k -> 49.9k
Connections:
- net LVGND: now also J4.3 (Pin_3), Q2.2 (S), R14.1, R16.2
- net SignalHV: now also R5.1, SigHV_TP1.1, U3.4
- net SignalLV: now also J4.4 (Pin_4), SignalLV1.1; no longer Q3.1 (G), R11.1
- net Con+ renamed LV+
- net LV+: now also D6.1 (K), J6.1 (Pin_1), J6.2 (Pin_2), J7.1 (Pin_1), J7.2 (Pin_2), R17.2
- net Con- renamed PreCon-
- net PreCon-: now also J6.4 (Pin_4)
- net Sense renamed Pre_Sense
- net Pre_Sense: now also J4.1 (Pin_1), J6.3 (Pin_3)
- new net: Con2.2 (A), R17.1
- new net GND: U1.29 (GND)
- new net MACon-: Con2.1 (K), D6.2 (A), J7.4 (Pin_4), Q2.3 (D)
- new net Mot_Arr_Sense: J4.2 (Pin_2), J7.3 (Pin_3), R14.2
- new net Mot_Arr_Signal: Q2.1 (G), R16.1
- new net PreSignal: Q3.1 (G), R11.1
Other:
- note added: "CAN CONN"
- note added: "CAN IC"
- note added: "Motor/Array Coil+"
- note added: "Motor/Array Coil-"
- note added: "Motor/Array Contactor Indicator LED"
- note added: "NUCLEO PWR Circuitry"
- note added: "Precharge Coil+"
- note added: "Precharge Coil-"
- note added: "Precharge Contactor Indicator LED"
- note added: "Signal LV, LVGND and Motor/Array and Precharge Sense for controls"
- note removed: "Coil+"
- note removed: "Coil-"
- note removed: "Contactor Driver Gate Signal and Contactor Sense Signal for controls"
- note removed: "Contactor Indicator LED"
- note removed: "Fan+"
- note removed: "Fan-"
- moved on the sheet: 12V_TP1, C1, C2, C3, C4, C5, Con1, D1, D2, D3, D4, D5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
