File: CAN.kicad_sch (KiCad schematic)
At the start: 17 parts, among them J8 CAN_IN, J9 CAN_OUT, U6 ADM3055E, U7 CDSOT23-T24CAN

Commit message: further schematic changes
Parts:
- renumbered J9 to J10, J8 to J9
Changed lines of the file:
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@@
 		(on_board yes)
 		(dnp no)
-		(property "Reference" "J9"
+		(property "Reference" "J10"
 			(at 221.742 92.9132 0)
 			(effects
@@
 			(project "ActivePrecharge"
 				(path "/b9847a31-2b3b-47ca-9561-fab506416f6d/a2982df7-4a65-4a2b-8298-6a7a639680dd"
-					(reference "J9")
+					(reference "J10")
 					(unit 1)
 				)
@@
 		(on_board yes)
 		(dnp no)
-		(property "Reference" "J8"
+		(property "Reference" "J9"
 			(at 221.7166 81.4832 0)
 			(effects
@@
 			(project "ActivePrecharge"
 				(path "/b9847a31-2b3b-47ca-9561-fab506416f6d/a2982df7-4a65-4a2b-8298-6a7a639680dd"
-					(reference "J8")
+					(reference "J9")
 					(unit 1)
 				)
